File: hw/pracka.brd (EAGLE design)
At the start: 109.2 x 86 mm, 100 parts, among them IC1 78L05Z, IC4 STM32F10XCXT6

Commit message: hardware fixes
Connections:
- net +3V3: now also SL4.1
- net GND: no longer SL4.1
- net L_ZBYTEK: now also TR6.A1
- net P_PUMP: no longer TR6.A1
Routing:
- net +3V3: track 301.1 -> 333.7 mm
- net P_PUMP: track 30.6 -> 25.0 mm
- net L_ZBYTEK: track 48.1 -> 52.1 mm
Other:
- board text added: "HW1.1"
Changed lines of the file:
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@@
 <grid distance="0.3175" unitdist="mm" unit="mm" style="lines" multiple="1" display="no" altdistance="0.15875" altunitdist="mm" altunit="mm"/>
 <layers>
-<layer number="1" name="Top" color="4" fill="1" visible="no" active="yes"/>
+<layer number="1" name="Top" color="4" fill="1" visible="yes" active="yes"/>
 <layer number="2" name="Route2" color="1" fill="3" visible="no" active="no"/>
 <layer number="3" name="Route3" color="4" fill="3" visible="no" active="no"/>
@@
 <layer number="14" name="Route14" color="1" fill="6" visible="no" active="no"/>
 <layer number="15" name="Route15" color="4" fill="6" visible="no" active="no"/>
-<layer number="16" name="Bottom" color="1" fill="1" visible="no" active="yes"/>
-<layer number="17" name="Pads" color="2" fill="1" visible="no" active="yes"/>
-<layer number="18" name="Vias" color="2" fill="1" visible="no" active="yes"/>
-<layer number="19" name="Unrouted" color="6" fill="1" visible="no" active="yes"/>
+<layer number="16" name="Bottom" color="1" fill="1" visible="yes" active="yes"/>
+<layer number="17" name="Pads" color="2" fill="1" visible="yes" active="yes"/>
+<layer number="18" name="Vias" color="2" fill="1" visible="yes" active="yes"/>
+<layer number="19" name="Unrouted" color="6" fill="1" visible="yes" active="yes"/>
 <layer number="20" name="Dimension" color="15" fill="1" visible="yes" active="yes"/>
 <layer number="21" name="tPlace" color="7" fill="1" visible="yes" active="yes"/>
-<layer number="22" name="bPlace" color="7" fill="1" visible="no" active="yes"/>
+<layer number="22" name="bPlace" color="7" fill="1" visible="yes" active="yes"/>
 <layer number="23" name="tOrigins" color="15" fill="1" visible="yes" active="yes"/>
-<layer number="24" name="bOrigins" color="15" fill="1" visible="no" active="yes"/>
+<layer number="24" name="bOrigins" color="15" fill="1" visible="yes" active="yes"/>
 <layer number="25" name="tNames" color="7" fill="1" visible="yes" active="yes"/>
-<layer number="26" name="bNames" color="7" fill="1" visible="no" active="yes"/>
+<layer number="26" name="bNames" color="7" fill="1" visible="yes" active="yes"/>
 <layer number="27" name="tValues" color="7" fill="1" visible="no" active="yes"/>
 <layer number="28" name="bValues" color="7" fill="1" visible="no" active="yes"/>
@@
 <text x="99.06" y="-2.2225" size="1.778" layer="102" rot="R270">DOOR LOCKED</text>
 <text x="105.0925" y="-2.54" size="1.778" layer="102" rot="R270">NEUTRAL</text>
+<text x="35.8775" y="56.8325" size="1.9304" layer="16" font="vector" ratio="21" rot="MR0">HW1.1</text>
 </plain>
 <attributes>
@@
 <contactref element="SL1" pad="1"/>
 <contactref element="SL3" pad="1"/>
-<contactref element="SL4" pad="1"/>
 <contactref element="C10" pad="2"/>
 <contactref element="U$1" pad="2"/>
@@
 <contactref element="TR5" pad="A2"/>
 <contactref element="R10" pad="2"/>
-<contactref element="TR6" pad="A1"/>
 <contactref element="X6" pad="1"/>
 <wire x1="59.69" y1="20.32" x2="63.5" y2="20.32" width="1.6764" layer="16"/>
@@
 <wire x1="69.85" y1="11.43" x2="71.12" y2="10.16" width="1.6764" layer="16"/>
 <wire x1="71.12" y1="10.16" x2="71.12" y2="5.715" width="1.6764" layer="16"/>
-<wire x1="68.58" y1="22.86" x2="64.77" y2="22.86" width="1.6764" layer="16"/>
-<wire x1="64.77" y1="22.86" x2="63.5" y2="21.59" width="1.6764" layer="16"/>
 <wire x1="63.5" y1="21.59" x2="63.5" y2="20.32" width="1.6764" layer="16"/>
 </signal>
@@
 <wire x1="78.74" y1="22.86" x2="78.74" y2="24.13" width="1.6764" layer="16"/>
 <wire x1="78.74" y1="24.13" x2="76.2" y2="26.67" width="1.6764" layer="16"/>
-<wire x1="76.2" y1="26.67" x2="60.96" y2="26.67" width="1.6764" layer="16"/>
+<wire x1="76.2" y1="26.67" x2="68.2625" y2="26.67" width="1.6764" layer="16"/>
+<wire x1="68.2625" y1="26.67" x2="60.96" y2="26.67" width="1.6764" layer="16"/>
 <wire x1="60.96" y1="26.67" x2="59.69" y2="25.4" width="1.6764" layer="16"/>
 <wire x1="59.69" y1="25.4" x2="59.69" y2="22.86" width="1.6764" layer="16"/>
@@
 <wire x1="96.0247" y1="26.4922" x2="97.155" y2="27.6225" width="0.4064" layer="16"/>
 <wire x1="97.155" y1="27.6225" x2="97.155" y2="31.4325" width="0.4064" layer="16"/>
+<contactref element="TR6" pad="A1"/>
+<wire x1="68.58" y1="22.86" x2="68.58" y2="26.3525" width="1.778" layer="16"/>
+<wire x1="68.58" y1="26.3525" x2="68.2625" y2="26.67" width="1.778" layer="16"/>
 </signal>
 <signal name="N$30">
@@
 <wire x1="70.6725" y1="63.37" x2="72.0725" y2="64.77" width="0.4064" layer="16"/>
 <via x="72.0725" y="64.77" extent="1-16" drill="0.5" diameter="1.27"/>
-<wire x1="72.0725" y1="64.77" x2="79.0575" y2="64.77" width="0.4064" layer="1"/>
-<via x="79.0575" y="64.77" extent="1-16" drill="0.5" diameter="1.27"/>
-<wire x1="79.0575" y1="64.77" x2="87.63" y2="64.77" width="0.4064" layer="16"/>
+<wire x1="72.0725" y1="64.77" x2="82.8675" y2="64.77" width="0.4064" layer="1"/>
+<via x="82.8675" y="64.77" extent="1-16" drill="0.5" diameter="1.27"/>
+<wire x1="82.8675" y1="64.77" x2="87.63" y2="64.77" width="0.4064" layer="16"/>
 <wire x1="87.63" y1="64.77" x2="89.2175" y2="63.1825" width="0.4064" layer="16"/>
 <wire x1="89.2175" y1="63.1825" x2="105.41" y2="63.1825" width="0.4064" layer="16"/>
@@
 <vertex x="55.88" y="67.945"/>
 </polygon>
+<contactref element="SL4" pad="1"/>
+<wire x1="78.4225" y1="81.28" x2="78.4225" y2="79.6925" width="0.4064" layer="16"/>
+<wire x1="78.4225" y1="79.6925" x2="77.1525" y2="78.4225" width="0.4064" layer="16"/>
+<wire x1="77.1525" y1="78.4225" x2="77.1525" y2="72.39" width="0.4064" layer="16"/>
+<wire x1="77.1525" y1="72.39" x2="76.835" y2="72.0725" width="0.4064" layer="16"/>
+<wire x1="76.835" y1="72.0725" x2="76.835" y2="59.69" width="0.4064" layer="16"/>
+<wire x1="76.835" y1="59.69" x2="77.47" y2="59.055" width="0.4064" layer="16"/>
+<wire x1="77.47" y1="59.055" x2="80.01" y2="59.055" width="0.4064" layer="16"/>
+<wire x1="80.01" y1="59.055" x2="82.8675" y2="61.9125" width="0.4064" layer="16"/>
+<wire x1="82.8675" y1="61.9125" x2="82.8675" y2="64.77" width="0.4064" layer="16"/>
 </signal>
 <signal name="N$39">
@@
 <wire x1="43.18" y1="69.345" x2="43.18" y2="71.755" width="0.4064" layer="16"/>
 </signal>
+<signal name="N$59">
+</signal>
+<signal name="N$62">
+</signal>
+<signal name="N$66">
+</signal>
 </signals>
