File: hw/pracka.sch (EAGLE design)
At the start: 100 parts, among them IC1 78L05Z, IC4 STM32F10XCXT6

Commit message: hardware fixes
Connections:
- net +3V3: now also SL4.1
- net GND: no longer SL4.1
- net L_ZBYTEK: now also TR6.A1
- net P_PUMP: no longer TR6.A1
Other:
- note added: "FAST motor"
- note added: "M"
- note added: "SLOW motor"
- note removed: "3x motor"
